File: PCB_v2/MicroMouse Power Subsystem project.kicad_sch (KiCad schematic)
At the start: 48 parts, among them IC1 CH224K, IC2 TPS61088RHLR, IC3 TPS63802DLAR, J1 USB_C_Receptacle_USB2.0, J2 Conn_01x02 (Battery), J3 Conn_02x16_Odd_Even, U2 BQ24074RGT

Commit message: Latest updates made with some footprints.
Parts:
- IC1: footprint SOP100P600X180-11N -> Library_3088:SOP100P600X180-11N; LCSC (none) -> C970725
- IC2: footprint RHL(R-PVQFN-N20)_1 -> Library_3088:RHL(R-PVQFN-N20)_1; LCSC (none) -> C87357
- IC3: footprint TPS63802DLAR -> Library_3088:TPS63802DLAR
- J1: value USB_C_Receptacle_USB2.0 -> GT-USB-7010ASV; symbol Connector:USB_C_Receptacle_USB2.0 -> Connector:USB_C_Receptacle_USB2.0_16P; LCSC (none) -> C2988369
- U2: footprint Package_DFN_QFN:VQFN-16-1EP_3x3mm_P0.5mm_EP1.6x1.6mm -> Library_3088:BQ24074RGTR
Connections:
- no-connect marks 10 -> 8
Changed lines of the file:
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@@
 	)
 	(no_connect
-		(at 41.275 49.53)
-	)
-	(no_connect
-		(at 41.275 52.07)
-	)
-	(no_connect
 		(at 154.305 52.07)
 	)
@@
 			)
 		)
-		(property "Footprint" "SOP100P600X180-11N"
+		(property "Footprint" "Library_3088:SOP100P600X180-11N"
 			(at 93.98 120.955 0)
 			(effects
@@
 			)
 		)
+		(property "LCSC" "C970725"
+			(at 67.31 26.035 0)
+			(effects
+				(font
+					(size 1.27 1.27)
+				)
+				(hide yes)
+			)
+		)
 		(pin "1"
 		)
@@
 			)
 		)
-		(property "Footprint" "TPS63802DLAR"
+		(property "Footprint" "Library_3088:TPS63802DLAR"
 			(at 243.84 122.225 0)
 			(effects
@@
 			)
 		)
-		(property "Footprint" "Package_DFN_QFN:VQFN-16-1EP_3x3mm_P0.5mm_EP1.6x1.6mm"
+		(property "Footprint" "Library_3088:BQ24074RGTR"
 			(at 161.925 50.8 0)
 			(effects
@@
 			)
 		)
-		(property "Footprint" "RHL(R-PVQFN-N20)_1"
+		(property "Footprint" "Library_3088:RHL(R-PVQFN-N20)_1"
 			(at 157.15 84.455 0)
 			(effects
@@
 			)
 		)
+		(property "LCSC" "C87357"
+			(at 72.39 116.205 90)
+			(effects
+				(font
+					(size 1.27 1.27)
+				)
+				(hide yes)
+			)
+		)
 		(pin "1"
 		)
@@
 	)
 	(symbol
-		(lib_id "Connector:USB_C_Receptacle_USB2.0")
+		(lib_id "Connector:USB_C_Receptacle_USB2.0_16P")
 		(at 26.035 36.83 0)
 		(unit 1)
@@
 		(fields_autoplaced yes)
 		(property "Reference" "J1"
-			(at 26.035 14.605 0)
+			(at 26.035 13.97 0)
 			(effects
 				(font
@@
 			)
 		)
-		(property "Value" "USB_C_Receptacle_USB2.0"
-			(at 26.035 17.145 0)
+		(property "Value" "GT-USB-7010ASV"
+			(at 26.035 16.51 0)
 			(effects
 				(font
@@
 			)
 		)
-		(property "Description" ""
+		(property "Description" "USB 2.0-only 16P Type-C Receptacle connector"
+			(at 26.035 36.83 0)
+			(effects
+				(font
+					(size 1.27 1.27)
+				)
+				(hide yes)
+			)
+		)
+		(property "LCSC" "C2988369"
 			(at 26.035 36.83 0)
 			(effects
@@
 					(size 1.27 1.27)
 				)
+				(hide yes)
 			)
 		)
@@
 		(pin "A7"
 		)
-		(pin "A8"
-		)
 		(pin "A9"
 		)
@@
 		(pin "B7"
 		)
-		(pin "B8"
-		)
 		(pin "B9"
 		)
 		(pin "S1"
 		)
+		(pin "B8"
+		)
+		(pin "A8"
+		)
 		(instances
