File: PCB_v2/PCB_v2.kicad_sch (KiCad schematic)
At the start: 31 parts, among them J1 Conn_02x16_Odd_Even, U1 DRV8833PWPR, U2 DRV8833PWPR, U3 INA219AIDCNR, U4 SIP32431DNP3-T1GE4, U5 SIP32431DNP3-T1GE4

Commit message: Initial commit added
Parts:
- removed C3: 0.01uF, Capacitor_SMD:C_0402_1005Metric_Pad0.74x0.62mm_HandSolder, symbol Device:C
- removed C6: 10uF, Capacitor_SMD:C_0402_1005Metric_Pad0.74x0.62mm_HandSolder, symbol Device:C
- added C11: 2.2uF, Capacitor_SMD:C_0603_1608Metric_Pad1.08x0.95mm_HandSolder, symbol Device:C
- added C12: 0.01uF, Capacitor_SMD:C_0805_2012Metric_Pad1.18x1.45mm_HandSolder, symbol Device:C
- C10, C7, C8, C9: footprint Capacitor_SMD:C_0402_1005Metric_Pad0.74x0.62mm_HandSolder -> Capacitor_SMD:C_1206_3216Metric_Pad1.33x1.80mm_HandSolder
- C2: value 2.2uF -> 10uF; LCSC (none) -> C13585
- C4: footprint Capacitor_SMD:C_0402_1005Metric_Pad0.74x0.62mm_HandSolder -> Capacitor_SMD:C_0805_2012Metric_Pad1.18x1.45mm_HandSolder; LCSC (none) -> C1710
- C5: footprint Capacitor_SMD:C_0402_1005Metric_Pad0.74x0.62mm_HandSolder -> Capacitor_SMD:C_0603_1608Metric_Pad1.08x0.95mm_HandSolder; LCSC (none) -> C23630
- R3: footprint Resistor_SMD:R_01005_0402Metric -> Resistor_SMD:R_0805_2012Metric_Pad1.20x1.40mm_HandSolder; LCSC (none) -> C175742
- R5, R8: footprint Library:RESCAXS80P320X160X60-8N -> Resistor_SMD:R_1206_3216Metric_Pad1.30x1.75mm_HandSolder; LCSC C1980 -> C17936
Connections:
- net 5V Out: now also C9.1, U5.4 (IN); no longer U5.3 (ON)
- net Battery: now also C2.1, C12.1
- net CTRL_EXT_LOAD2: now also U5.3 (ON); no longer C9.1, U5.4 (IN)
- net GND: now also C11.2
- net at U1.11 (VCP): now also C12.2
- net at U1.14 (VINT): now also C11.1; no longer C2.1
Other:
- note added: "0.15 close enough to 0.16"
- note added: "done with footprints EXCULDIING test points"
- note removed: "Do I connect ON/OFF to vcc"
- note removed: "ENSURE THE IN AND OUT ARE CONNECTED CORRECTLY"
- moved on the sheet: C7, C9
